File: secukey.kicad_sch (KiCad schematic)
At the start: 44 parts, among them SW4 TS-1185-W-4P-H1.8-160, SW5 TS-1185-W-4P-H1.8-160, SW6 TS-1185-W-4P-H1.8-160, U2 RP2350A, U3 NCP1117-3.3_SOT223, U4 W25Q128JVS, U5 ABM8-272-T3_C20625731, U6 SM03B-SRSS-TB, U7 ATECC608A-MAHDA-T

Commit message: rearrange the placement for power route
Connections:
- net GND: now also SW4.1; no longer SW4.2
- net at SW4.3: no longer R14.1
- net at SW4.4: now also R14.1
Other:
- moved on the sheet: SW4
Changed lines of the file:
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@@
 	)
 	(no_connect
-		(at 275.59 106.68)
-	)
-	(no_connect
 		(at 209.55 55.88)
 	)
@@
 	)
 	(no_connect
-		(at 280.67 96.52)
-	)
-	(no_connect
 		(at 209.55 101.6)
 	)
@@
 	)
 	(no_connect
+		(at 276.86 102.87)
+	)
+	(no_connect
 		(at 128.27 132.08)
 	)
 	(no_connect
+		(at 266.7 107.95)
+	)
+	(no_connect
 		(at 209.55 60.96)
 	)
@@
 	(wire
 		(pts
-			(xy 275.59 93.98) (xy 275.59 96.52)
+			(xy 207.01 109.22) (xy 209.55 109.22)
 		)
 		(stroke
@@
 	(wire
 		(pts
-			(xy 207.01 109.22) (xy 209.55 109.22)
+			(xy 45.72 72.39) (xy 45.72 74.93)
 		)
 		(stroke
@@
 	(wire
 		(pts
-			(xy 45.72 72.39) (xy 45.72 74.93)
+			(xy 276.86 107.95) (xy 281.94 107.95)
 		)
 		(stroke
@@
 	(wire
 		(pts
-			(xy 271.78 83.82) (xy 270.51 83.82)
+			(xy 261.62 102.87) (xy 261.62 106.68)
 		)
 		(stroke
@@
 	(wire
 		(pts
-			(xy 260.35 55.88) (xy 262.89 55.88)
+			(xy 271.78 83.82) (xy 270.51 83.82)
 		)
 		(stroke
@@
 	(wire
 		(pts
-			(xy 271.78 86.36) (xy 270.51 86.36)
+			(xy 260.35 55.88) (xy 262.89 55.88)
 		)
 		(stroke
@@
 	(wire
 		(pts
-			(xy 270.51 93.98) (xy 275.59 93.98)
+			(xy 271.78 86.36) (xy 270.51 86.36)
 		)
 		(stroke
@@
 	(wire
 		(pts
+			(xy 281.94 107.95) (xy 281.94 93.98)
+		)
+		(stroke
+			(width 0)
+			(type default)
+		)
+	)
+	(wire
+		(pts
 			(xy 16.51 87.63) (xy 27.94 87.63)
 		)
@@
 	(wire
 		(pts
-			(xy 280.67 106.68) (xy 280.67 109.22)
+			(xy 143.51 64.77) (xy 140.97 64.77)
 		)
 		(stroke
@@
 	(wire
 		(pts
-			(xy 143.51 64.77) (xy 140.97 64.77)
+			(xy 91.44 62.23) (xy 91.44 64.77)
 		)
 		(stroke
@@
 	(wire
 		(pts
-			(xy 91.44 62.23) (xy 91.44 64.77)
+			(xy 57.15 72.39) (xy 57.15 74.93)
 		)
 		(stroke
@@
 	(wire
 		(pts
-			(xy 57.15 72.39) (xy 57.15 74.93)
+			(xy 121.92 46.99) (xy 121.92 48.26)
 		)
 		(stroke
@@
 	(wire
 		(pts
-			(xy 121.92 46.99) (xy 121.92 48.26)
+			(xy 139.7 45.72) (xy 139.7 46.99)
 		)
 		(stroke
@@
 	(wire
 		(pts
-			(xy 139.7 45.72) (xy 139.7 46.99)
+			(xy 281.94 93.98) (xy 270.51 93.98)
 		)
 		(stroke
@@
 	(wire
 		(pts
+			(xy 266.7 102.87) (xy 261.62 102.87)
+		)
+		(stroke
+			(width 0)
+			(type default)
+		)
+	)
+	(wire
+		(pts
 			(xy 49.53 181.61) (xy 44.45 181.61)
 		)
@@
 	(symbol
 		(lib_id "EasyEDA:TS-1185-W-4P-H1.8-160")
-		(at 279.4 101.6 270)
+		(at 271.78 104.14 0)
 		(unit 1)
 		(body_style 1)
@@
 		(fields_autoplaced yes)
 		(property "Reference" "SW4"
-			(at 281.94 100.3299 90)
+			(at 271.78 97.79 0)
 			(show_name no)
 			(do_not_autoplace no)
@@
 					(size 1.27 1.27)
 				)
-				(justify left)
 			)
 		)
 		(property "Value" "TS-1185-W-4P-H1.8-160"
-			(at 281.94 102.8699 90)
+			(at 271.78 100.33 0)
 			(show_name no)
 			(do_not_autoplace no)
@@
 					(size 1.27 1.27)
 				)
-				(justify left)
 			)
 		)
 		(property "Footprint" "EasyEDA:SW-SMD_4P-L3.5-W3.0-P1.50-LS4.7"
-			(at 267.97 101.6 0)
+			(at 271.78 115.57 0)
 			(hide yes)
 			(show_name no)
@@
 		)
 		(property "Datasheet" "https://www.lcsc.com/datasheet/C51927445.pdf"
-			(at 265.43 101.6 0)
+			(at 271.78 118.11 0)
 			(hide yes)
 			(show_name no)
@@
 		)
 		(property "Description" ""
-			(at 279.4 101.6 0)
+			(at 271.78 104.14 0)
 			(hide yes)
 			(show_name no)
@@
 		)
 		(property "Manufacturer" "CAX(创都)"
-			(at 262.89 101.6 0)
+			(at 271.78 120.65 0)
 			(hide yes)
 			(show_name no)
@@
 		)
 		(property "MPN" "TS-1185-W-4P-H1.8-160"
-			(at 260.35 101.6 0)
+			(at 271.78 123.19 0)
 			(hide yes)
 			(show_name no)
@@
 		)
 		(property "LCSC Part" "C51927445"
-			(at 257.81 101.6 0)
+			(at 271.78 125.73 0)
 			(hide yes)
 			(show_name no)
@@
 	(symbol
 		(lib_id "power:GND")
-		(at 280.67 109.22 0)
+		(at 261.62 106.68 0)
 		(unit 1)
 		(body_style 1)
@@
 		(fields_autoplaced yes)
 		(property "Reference" "#PWR023"
-			(at 280.67 115.57 0)
+			(at 261.62 113.03 0)
 			(hide yes)
 			(show_name no)
@@
 		)
 		(property "Value" "GND"
-			(at 280.67 114.3 0)
+			(at 261.62 111.76 0)
 			(show_name no)
 			(do_not_autoplace no)
@@
 		)
 		(property "Footprint" ""
-			(at 280.67 109.22 0)
+			(at 261.62 106.68 0)
 			(hide yes)
 			(show_name no)
@@
 		)
 		(property "Datasheet" ""
-			(at 280.67 109.22 0)
+			(at 261.62 106.68 0)
 			(hide yes)
 			(show_name no)
@@
 		)
 		(property "Description" "Power symbol creates a global label with name \"GND\" , ground"
-			(at 280.67 109.22 0)
+			(at 261.62 106.68 0)
 			(hide yes)
 			(show_name no)

Commit message: adding ref
Parts:
- removed C1, C17, C2, C3: 4.7u, Capacitor_SMD:C_0402_1005Metric, symbol Device:C
- removed C10, C11, C12, C13, C14, C15, C16, C18, C6, C7, C8, C9: 100n, Capacitor_SMD:C_0402_1005Metric, symbol Device:C
- removed C19, C20: 15p, Capacitor_SMD:C_0402_1005Metric, symbol Device:C
- removed C21: 100nF, Capacitor_SMD:C_0402_1005Metric, symbol Device:C
- removed C4, C5: 10u, Capacitor_SMD:C_0402_1005Metric, symbol Device:C
- removed R1: 33Ω, Resistor_SMD:R_0402_1005Metric, symbol Device:R
- removed R10, R9: 4,7kΩ, Resistor_SMD:R_0402_1005Metric, symbol Device:R
- removed R13: 10kΩ, Resistor_SMD:R_0402_1005Metric, symbol Device:R
- removed R14, R7, R8: 1k, Resistor_SMD:R_0402_1005Metric, symbol Device:R
- added C1, C2: FCC0805N150J500BT, EasyEDA:C0805, symbol EasyEDA:FCC0805N150J500BT
- added C22, C23, C24, C25, C26, C27, C28, C29, C30, C31, C32, C33, C34, C35, C36, C37: CC0402KRX7R5BB104, EasyEDA:C0402, symbol EasyEDA:CC0402KRX7R5BB104
- added C4, C5, C6: CL21A475KBQNNNE, EasyEDA:C0805, symbol EasyEDA:CL21A475KBQNNNE
- added R1: RC0805JR-0710KL, EasyEDA:R0805, symbol EasyEDA:RC0805JR-0710KL
- added R10, R13, R14: RC0805JR-071KL, EasyEDA:R0805, symbol EasyEDA:RC0805JR-071KL
- added R2: 0805W8J0330T5E, EasyEDA:R0805, symbol EasyEDA:0805W8J0330T5E
- added R3, R9: 0805W8F4701T5E, EasyEDA:R0805, symbol EasyEDA:0805W8F4701T5E
Connections:
- net +1V1: now also C31.1, C32.1, C33.1, C5.1
- net +3.3V: now also C22.1, C23.1, C24.1, C25.1, C26.1, C27.1, C28.1, C29.1, C30.1, C34.1, C35.2, C37.1, C6.1, R1.2, R2.1, R3.2, R9.2
- net GND: now also C1.2, C2.1, C22.2, C23.2, C24.2, C25.2, C26.2, C27.2, C28.2, C29.2, C30.2, C31.2, C32.2, C33.2, C34.2, C35.1, C36.2, C37.2, C4.2, C5.2, C6.2
- net RP2350B_GPIO2: now also R1.1
- net RP2350B_GPIO4: now also R9.1
- net RP2350B_GPIO5: now also R3.1
- net RP2350B_QSPI_SS: now also R10.2
- net RP2350B_VREG-AVDD: now also C4.1, R2.2
- net RP2350B_XIN: now also C2.2
- net RP2350B_XOUT: now also R13.2
- net VBUS: now also C36.1
- net at SW4.4: now also R14.2
- net at U2.26 (RUN): now also R14.1
- net at SW6.3: now also R10.1
- net at U5.3: now also C1.1, R13.1

Commit message: adding made placement
Parts:
- removed R11, R12: 27, Resistor_SMD:R_0402_1005Metric, symbol Device:R
- removed R6: 0, Resistor_SMD:R_0402_1005Metric, symbol Device:R
- added R6, R8: FRC0805F27R0TS, EasyEDA:R0805, symbol EasyEDA:FRC0805F27R0TS
- added R7: 0805W8F0000T5E, EasyEDA:R0805, symbol EasyEDA:0805W8F0000T5E
Connections:
- net GND: now also U7.1 (NC), U7.2 (NC), U7.3 (NC), U7.7 (NC)
- net RP2350B_GPIO4: now also U2.7 (GPIO4)
- net RP2350B_GPIO5: now also U2.8 (GPIO5)
- net RP2350B_QSPI_SD0: now also U4.5 (DI/IO_{0})
- net RP2350B_QSPI_SD1: now also U4.2 (DO/IO_{1})
- net RP2350B_QSPI_SD2: now also U4.3 (~{WP}/IO_{2})
- net RP2350B_QSPI_SD3: now also U4.7 (~{HOLD}/~{RESET}/IO_{3})
- net RP2350B_QSPI_SS: now also R7.1
- net USB_D+: now also R8.2
- net USB_D-: now also R6.2
- net at U2.51 (USB_DM): now also R8.1
- net at R4.2, R5.2, U4.1 (~{CS}): now also R7.2
- net at U2.52 (USB_DP): now also R6.1
- no-connect marks 38 -> 32
